Commit message: added navigation stack

File: urdf/color_properties.xacro (robot description, xacro)
@@ -3,4 +3,7 @@
     <material name="green">
         <color rgba="0 1 0 1"/>
+    </material>
+    <material name="red">
+        <color rgba="1 0 0 1"/>
     </material>
     <material name="black">

File: urdf/manipulator.urdf (robot description, URDF)
Before this commit: robot manipulator_complete, 11 links, 10 joints
Links:
- added link imu_link
- added link laser_scanner, mass 0.002; collision box size=0.02 0.02 0.02; visual box size=0.02 0.02 0.02
- link arm_base: geometry collision mesh filename=package://mobile_manipulator_robot/meshes/arm_base.stl; visual mesh filename=package://mobile_manipulator_robot/meshes/arm_base.stl
- link bicep: geometry collision mesh filename=package://mobile_manipulator_robot/meshes/bicep.stl; visual mesh filename=package://mobile_manipulator_robot/meshes/bicep.stl
- link bottom_wrist: geometry collision mesh filename=package://mobile_manipulator_robot/meshes/wrist.stl; visual mesh filename=package://mobile_manipulator_robot/meshes/wrist.stl
- link elbow: geometry collision mesh filename=package://mobile_manipulator_robot/meshes/elbow.stl; visual mesh filename=package://mobile_manipulator_robot/meshes/elbow.stl
- link top_wrist: geometry collision mesh filename=package://mobile_manipulator_robot/meshes/wrist.stl; visual mesh filename=package://mobile_manipulator_robot/meshes/wrist.stl
Joints:
- added joint imu_joint: type fixed, parent base_link, child imu_link, origin xyz=-0.032 0 0.068 rpy=0 0 0
- added joint laser_scan_joint: type fixed, parent base_link, child laser_scanner, origin xyz=0.32 0 0.28 rpy=0 0 0
