Commit message: Add files via upload

File: urdf/manipulator.urdf (robot description, URDF)
Before this commit: robot manipulator_complete, 13 links, 12 joints
Links:
- added link camera_link, mass 1e-5; collision box size=0.02 0.02 0.02; visual box size=0.02 0.02 0.02
- added link camera_link_optical
- added link vacuum_gripper, mass 0.0001; visual cylinder length=0.01 radius=0.005
- added link vacuum_gripper1, mass 0.0001; visual cylinder length=0.01 radius=0.005
- added link vacuum_gripper10, mass 0.0001; visual cylinder length=0.01 radius=0.005
- added link vacuum_gripper11, mass 0.0001; visual cylinder length=0.01 radius=0.005
- added link vacuum_gripper12, mass 0.0001; visual cylinder length=0.01 radius=0.005
- added link vacuum_gripper2, mass 0.0001; visual cylinder length=0.01 radius=0.005
- added link vacuum_gripper3, mass 0.0001; visual cylinder length=0.01 radius=0.005
- added link vacuum_gripper4, mass 0.0001; visual cylinder length=0.01 radius=0.005
- added link vacuum_gripper5, mass 0.0001; visual cylinder length=0.01 radius=0.005
- added link vacuum_gripper6, mass 0.0001; visual cylinder length=0.01 radius=0.005
- added link vacuum_gripper7, mass 0.0001; visual cylinder length=0.01 radius=0.005
- added link vacuum_gripper8, mass 0.0001; visual cylinder length=0.01 radius=0.005
- added link vacuum_gripper9, mass 0.0001; visual cylinder length=0.01 radius=0.005
- added link vacuum_gripper_base, mass 0.0001; collision cylinder length=0.006 radius=0.04; visual cylinder length=0.02 radius=0.04
Joints:
- added joint camera_joint: type fixed, parent vacuum_gripper_base, child camera_link, origin xyz=-0.05 0.0 0.0 rpy=3.14 -1.57 0
- added joint camera_optical_joint: type fixed, parent camera_link, child camera_link_optical, origin xyz=0 0 0 rpy=0 0 0
- added joint gripper_joint: type revolute, parent vacuum_gripper_base, child vacuum_gripper, origin xyz=0.02 0.015 0.03 rpy=0 0 0, limit lower=0 upper=0 effort=50 velocity=50
- added joint gripper_joint1: type revolute, parent vacuum_gripper_base, child vacuum_gripper1, origin xyz=0.02 -0.015 0.03 rpy=0 0 0, limit lower=0 upper=0 effort=50 velocity=50
- added joint gripper_joint10: type revolute, parent vacuum_gripper_base, child vacuum_gripper10, origin xyz=-0.02 0.015 0.03 rpy=0 0 0, limit lower=0 upper=0 effort=50 velocity=50
- added joint gripper_joint11: type revolute, parent vacuum_gripper_base, child vacuum_gripper11, origin xyz=-0.02 -0.015 0.03 rpy=0 0 0, limit lower=0 upper=0 effort=50 velocity=50
- added joint gripper_joint12: type revolute, parent vacuum_gripper_base, child vacuum_gripper12, origin xyz=-0.01 0.015 0.03 rpy=0 0 0, limit lower=0 upper=0 effort=50 velocity=50
- added joint gripper_joint2: type revolute, parent vacuum_gripper_base, child vacuum_gripper2, origin xyz=-0.02 0 0.03 rpy=0 0 0, limit lower=0 upper=0 effort=50 velocity=50
- added joint gripper_joint3: type revolute, parent vacuum_gripper_base, child vacuum_gripper3, origin xyz=0 0 0.03 rpy=0 0 0, limit lower=0 upper=0 effort=50 velocity=50
- added joint gripper_joint4: type revolute, parent vacuum_gripper_base, child vacuum_gripper4, origin xyz=0.0 0.015 0.03 rpy=0 0 0, limit lower=0 upper=0 effort=50 velocity=50
- added joint gripper_joint5: type revolute, parent vacuum_gripper_base, child vacuum_gripper5, origin xyz=0.0 -0.015 0.03 rpy=0 0 0, limit lower=0 upper=0 effort=50 velocity=50
- added joint gripper_joint6: type revolute, parent vacuum_gripper_base, child vacuum_gripper6, origin xyz=0.01 -0.015 0.03 rpy=0 0 0, limit lower=0 upper=0 effort=50 velocity=50
- added joint gripper_joint7: type revolute, parent vacuum_gripper_base, child vacuum_gripper7, origin xyz=0.01 0.015 0.03 rpy=0 0 0, limit lower=0 upper=0 effort=50 velocity=50
- added joint gripper_joint8: type revolute, parent vacuum_gripper_base, child vacuum_gripper8, origin xyz=-0.01 -0.015 0.03 rpy=0 0 0, limit lower=0 upper=0 effort=50 velocity=50
- added joint gripper_joint9: type revolute, parent vacuum_gripper_base, child vacuum_gripper9, origin xyz=0.02 0.0 0.03 rpy=0 0 0, limit lower=0 upper=0 effort=50 velocity=50
- added joint vacuum_base_joint: type fixed, parent top_wrist, child vacuum_gripper_base, origin xyz=0.0 0 0.14 rpy=0 0 0
